File: EA3_V3_kicad.kicad_pcb (KiCad board)
At the start: 2 copper layers, 4 parts

Commit message: 3D BFP
Parts:
- added REF**: SOT343, BFP640:SOT343, F.Cu at (138.5, 89.9)
Changed lines of the file:
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@@
       (stroke (width 0.01) (type solid)) (fill solid) (layer "B.Mask"))
+  )
+  (footprint "BFP640:SOT343" (layer "F.Cu")
+    (at 138.5 89.9)
+    (attr smd)
+    (fp_text reference "REF**" (at 1.691281 0.060045 180) (layer "F.SilkS") hide
+        (effects (font (size 0.315198 0.315198) (thickness 0.0788)))
+    )
+    (fp_text value "SOT343" (at 0.145133 -0.005005) (layer "F.Fab") hide
+        (effects (font (size 0.315245 0.315245) (thickness 0.078811)))
+    )
+    (pad "1" smd rect (at -0.65 0.8) (size 0.6 0.8) (layers "F.Cu" "F.Paste" "F.Mask")
+      (solder_mask_margin 0.102))
+    (pad "2" smd rect (at 0.5 0.8) (size 0.9 0.8) (layers "F.Cu" "F.Paste" "F.Mask")
+      (solder_mask_margin 0.102))
+    (pad "3" smd rect (at 0.65 -0.8) (size 0.6 0.8) (layers "F.Cu" "F.Paste" "F.Mask")
+      (solder_mask_margin 0.102))
+    (pad "4" smd rect (at -0.65 -0.8) (size 0.6 0.8) (layers "F.Cu" "F.Paste" "F.Mask")
+      (solder_mask_margin 0.102))
+    (model "D:/Downloads/BFP640/BFP640.step"
+      (offset (xyz 0 0 0))
+      (scale (xyz 1 1 1))
+      (rotate (xyz -90 0 0))
+    )
   )
   (footprint "LOGO" (layer "F.Cu")
